Commit message: Add robot description file for SO101 follower with detailed URDF structure
- Created `robot_description.txt` containing the URDF for the SO101 follower robot.
- The file includes definitions for links, joints, materials, and visual/collision geometries.
- Generated using xacro from the Onshape CAD model, ensuring accurate representation of the robot's physical structure.

File: hiwonder_ros2/so101_follower_description/urdf/so101_follower.urdf.xacro (robot description, xacro)
@@ -1,13 +1,7 @@
-<?xml version='1.0' encoding='utf-8'?>
+<?xml version="1.0" encoding="utf-8"?>
 <!-- Generated using onshape-to-robot -->
 <!-- Onshape https://cad.onshape.com/documents/7715cc284bb430fe6dab4ffd/w/4fd0791b683777b02f8d975a/e/826c553ede3b7592eb9ca800 -->
-<robot name="so101_follower" xmlns:xacro="http://www.ros.org/wiki/xacro">
-  <!-- World Link -->
-  <link name="world"/>
-  <joint name="world_to_base" type="fixed">
-    <parent link="world"/>
-    <child link="base_link"/>
-    <origin xyz="0 0 0" rpy="0 0 0"/>
-  </joint>
+<!-- Derived from so101_new_calib.urdf: adds wrist camera mount + wrist camera (Hex-Nut 32x32 UVC module form factor) -->
+<robot name="so101_new_calib_camera">
   <!-- Materials -->
   <material name="3d_printed">
@@ -17,15 +11,14 @@
     <color rgba="0.1 0.1 0.1 1.0"/>
   </material>
-  <!-- Hard-coded calibrated limits (matching your calibration file) -->
   <!-- Link base -->
   <link name="base_link">
     <inertial>
-      <origin xyz="0.020739 0.00204287 0.065966" rpy="0 0 0"/>
+      <origin xyz="0.0137179 -5.19711e-05 0.0334843" rpy="0 0 0"/>
       <mass value="0.147"/>
-      <inertia ixx="0.000136117" ixy="4.59787e-07" ixz="9.75275e-08" iyy="0.000114686" iyz="-4.97151e-06" izz="0.000130364"/>
+      <inertia ixx="0.000114686" ixy="-4.59787e-07" ixz="4.97151e-06" iyy="0.000136117" iyz="9.75275e-08" izz="0.000130364"/>
     </inertial>
     <!-- Part base_motor_holder_so101_v1 -->
     <visual>
-      <origin xyz="0.0206915 0.0221255 0.0300817" rpy="1.5708 -1.23909e-16 2.33147e-15"/>
+      <origin xyz="-0.00636471 -9.94414e-05 -0.0024" rpy="1.5708 -1.67685e-15 1.5708"/>
       <geometry>
         <mesh filename="package://so101_follower_description/meshes/base_motor_holder_so101_v1.stl"/>
@@ -34,5 +27,5 @@
     </visual>
     <collision>
-      <origin xyz="0.0206915 0.0221255 0.0300817" rpy="1.5708 -1.23909e-16 2.33147e-15"/>
+      <origin xyz="-0.00636471 -9.94414e-05 -0.0024" rpy="1.5708 -1.67685e-15 1.5708"/>
       <geometry>
         <mesh filename="package://so101_follower_description/meshes/base_motor_holder_so101_v1.stl"/>
@@ -41,5 +34,5 @@
     <!-- Part base_so101_v2 -->
     <visual>
-      <origin xyz="0.0207909 0.0221255 0.0300817" rpy="1.5708 -0 0"/>
+      <origin xyz="-0.00636471 -8.97657e-09 -0.0024" rpy="1.5708 -2.78073e-29 1.5708"/>
       <geometry>
         <mesh filename="package://so101_follower_description/meshes/base_so101_v2.stl"/>
@@ -48,5 +41,5 @@
     </visual>
     <collision>
-      <origin xyz="0.0207909 0.0221255 0.0300817" rpy="1.5708 -0 0"/>
+      <origin xyz="-0.00636471 -8.97657e-09 -0.0024" rpy="1.5708 -2.78073e-29 1.5708"/>
       <geometry>
         <mesh filename="package://so101_follower_description/meshes/base_so101_v2.stl"/>
@@ -55,12 +48,12 @@
     <!-- Part sts3215_03a_v1 -->
     <visual>
-      <origin xyz="0.0207909 -0.0105745 0.0761817" rpy="-2.20282e-15 2.77556e-17 -1.5708"/>
-      <geometry>
-        <mesh filename="package://so101_follower_description/meshes/sts3215_03a_v1.stl"/>
-      </geometry>
-      <material name="sts3215"/>
-    </visual>
-    <collision>
-      <origin xyz="0.0207909 -0.0105745 0.0761817" rpy="-2.20282e-15 2.77556e-17 -1.5708"/>
+      <origin xyz="0.0263353 -8.97657e-09 0.0437" rpy="-8.21148e-16 7.84513e-18 1.249e-15"/>
+      <geometry>
+        <mesh filename="package://so101_follower_description/meshes/sts3215_03a_v1.stl"/>
+      </geometry>
+      <material name="sts3215"/>
+    </visual>
+    <collision>
+      <origin xyz="0.0263353 -8.97657e-09 0.0437" rpy="-8.21148e-16 7.84513e-18 1.249e-15"/>
       <geometry>
         <mesh filename="package://so101_follower_description/meshes/sts3215_03a_v1.stl"/>
@@ -69,5 +62,5 @@
     <!-- Part waveshare_mounting_plate_so101_v2 -->
     <visual>
-      <origin xyz="0.0205915 0.0467435 0.0798817" rpy="1.5708 -1.21716e-14 2.33147e-15"/>
+      <origin xyz="-0.0309827 -0.000199441 0.0474" rpy="1.5708 -1.35493e-14 1.5708"/>
       <geometry>
         <mesh filename="package://so101_follower_description/meshes/waveshare_mounting_plate_so101_v2.stl"/>
@@ -76,5 +69,5 @@
     </visual>
     <collision>
-      <origin xyz="0.0205915 0.0467435 0.0798817" rpy="1.5708 -1.21716e-14 2.33147e-15"/>
+      <origin xyz="-0.0309827 -0.000199441 0.0474" rpy="1.5708 -1.35493e-14 1.5708"/>
       <geometry>
         <mesh filename="package://so101_follower_description/meshes/waveshare_mounting_plate_so101_v2.stl"/>
@@ -119,5 +112,5 @@
     <!-- Part rotation_pitch_so101_v1 -->
     <visual>
-      <origin xyz="0.0122008 2.22413e-05 0.0464" rpy="-1.5708 -0 0"/>
+      <origin xyz="0.0122008 2.22413e-05 0.0464" rpy="-1.5708 2.35221e-33 0"/>
       <geometry>
         <mesh filename="package://so101_follower_description/meshes/rotation_pitch_so101_v1.stl"/>
@@ -126,5 +119,5 @@
     </visual>
     <collision>
-      <origin xyz="0.0122008 2.22413e-05 0.0464" rpy="-1.5708 -0 0"/>
+      <origin xyz="0.0122008 2.22413e-05 0.0464" rpy="-1.5708 2.35221e-33 0"/>
       <geometry>
         <mesh filename="package://so101_follower_description/meshes/rotation_pitch_so101_v1.stl"/>
@@ -141,12 +134,12 @@
     <!-- Part sts3215_03a_v1_3 -->
     <visual>
-      <origin xyz="-0.11257 -0.0155 0.0187" rpy="-3.14159 -6.8695e-16 -1.5708"/>
-      <geometry>
-        <mesh filename="package://so101_follower_description/meshes/sts3215_03a_v1.stl"/>
-      </geometry>
-      <material name="sts3215"/>
-    </visual>
-    <collision>
-      <origin xyz="-0.11257 -0.0155 0.0187" rpy="-3.14159 -6.8695e-16 -1.5708"/>
+      <origin xyz="-0.11257 -0.0155 0.0187" rpy="-3.14159 -5.27356e-16 -1.5708"/>
+      <geometry>
+        <mesh filename="package://so101_follower_description/meshes/sts3215_03a_v1.stl"/>
+      </geometry>
+      <material name="sts3215"/>
+    </visual>
+    <collision>
+      <origin xyz="-0.11257 -0.0155 0.0187" rpy="-3.14159 -5.27356e-16 -1.5708"/>
       <geometry>
         <mesh filename="package://so101_follower_description/meshes/sts3215_03a_v1.stl"/>
@@ -155,5 +148,5 @@
     <!-- Part upper_arm_so101_v1 -->
     <visual>
-      <origin xyz="-0.065085 0.012 0.0182" rpy="3.14159 -9.35612e-32 0"/>
+      <origin xyz="-0.065085 0.012 0.0182" rpy="3.14159 -0 -1.30911e-30"/>
       <geometry>
         <mesh filename="package://so101_follower_description/meshes/upper_arm_so101_v1.stl"/>
@@ -162,5 +155,5 @@
     </visual>
     <collision>
-      <origin xyz="-0.065085 0.012 0.0182" rpy="3.14159 -9.35612e-32 0"/>
+      <origin xyz="-0.065085 0.012 0.0182" rpy="3.14159 -0 -1.30911e-30"/>
       <geometry>
         <mesh filename="package://so101_follower_description/meshes/upper_arm_so101_v1.stl"/>
@@ -177,5 +170,5 @@
     <!-- Part under_arm_so101_v1 -->
     <visual>
-      <origin xyz="-0.0648499 -0.032 0.0182" rpy="-3.14159 -0 3.9443e-31"/>
+      <origin xyz="-0.0648499 -0.032 0.0182" rpy="3.14159 -0 6.67202e-31"/>
       <geometry>
         <mesh filename="package://so101_follower_description/meshes/under_arm_so101_v1.stl"/>
@@ -184,5 +177,5 @@
     </visual>
     <collision>
-      <origin xyz="-0.0648499 -0.032 0.0182" rpy="-3.14159 -0 3.9443e-31"/>
+      <origin xyz="-0.0648499 -0.032 0.0182" rpy="3.14159 -0 6.67202e-31"/>
       <geometry>
         <mesh filename="package://so101_follower_description/meshes/under_arm_so101_v1.stl"/>
@@ -191,5 +184,5 @@
     <!-- Part motor_holder_so101_wrist_v1 -->
     <visual>
-      <origin xyz="-0.0648499 -0.032 0.018" rpy="-3.14159 4.73317e-30 7.88861e-31"/>
+      <origin xyz="-0.0648499 -0.032 0.018" rpy="-3.14159 -2.55351e-15 -1.83387e-30"/>
       <geometry>
         <mesh filename="package://so101_follower_description/meshes/motor_holder_so101_wrist_v1.stl"/>
@@ -198,5 +191,5 @@
     </visual>
     <collision>
-      <origin xyz="-0.0648499 -0.032 0.018" rpy="-3.14159 4.73317e-30 7.88861e-31"/>
+      <origin xyz="-0.0648499 -0.032 0.018" rpy="-3.14159 -2.55351e-15 -1.83387e-30"/>
       <geometry>
         <mesh filename="package://so101_follower_description/meshes/motor_holder_so101_wrist_v1.stl"/>
@@ -205,12 +198,12 @@
     <!-- Part sts3215_03a_v1_4 -->
     <visual>
-      <origin xyz="-0.1224 0.0052 0.0187" rpy="-3.14159 -3.58047e-15 -3.14159"/>
-      <geometry>
-        <mesh filename="package://so101_follower_description/meshes/sts3215_03a_v1.stl"/>
-      </geometry>
-      <material name="sts3215"/>
-    </visual>
-    <collision>
-      <origin xyz="-0.1224 0.0052 0.0187" rpy="-3.14159 -3.58047e-15 -3.14159"/>
+      <origin xyz="-0.1224 0.0052 0.0187" rpy="-3.14159 -7.88861e-31 -3.14159"/>
+      <geometry>
+        <mesh filename="package://so101_follower_description/meshes/sts3215_03a_v1.stl"/>
+      </geometry>
+      <material name="sts3215"/>
+    </visual>
+    <collision>
+      <origin xyz="-0.1224 0.0052 0.0187" rpy="-3.14159 -7.88861e-31 -3.14159"/>
       <geometry>
         <mesh filename="package://so101_follower_description/meshes/sts3215_03a_v1.stl"/>
@@ -227,5 +220,5 @@
     <!-- Part sts3215_03a_no_horn_v1 -->
     <visual>
-      <origin xyz="5.55112e-17 -0.0424 0.0306" rpy="1.5708 1.5708 0"/>
+      <origin xyz="8.32667e-17 -0.0424 0.0306" rpy="1.5708 1.5708 0"/>
       <geometry>
         <mesh filename="package://so101_follower_description/meshes/sts3215_03a_no_horn_v1.stl"/>
@@ -234,5 +227,5 @@
     </visual>
     <collision>
-      <origin xyz="5.55112e-17 -0.0424 0.0306" rpy="1.5708 1.5708 0"/>
+      <origin xyz="8.32667e-17 -0.0424 0.0306" rpy="1.5708 1.5708 0"/>
       <geometry>
         <mesh filename="package://so101_follower_description/meshes/sts3215_03a_no_horn_v1.stl"/>
@@ -263,12 +256,12 @@
     <!-- Part sts3215_03a_v1_5 -->
     <visual>
-      <origin xyz="0.0077 0.0001 -0.0234" rpy="-1.5708 -5.55112e-17 -1.38213e-14"/>
-      <geometry>
-        <mesh filename="package://so101_follower_description/meshes/sts3215_03a_v1.stl"/>
-      </geometry>
-      <material name="sts3215"/>
-    </visual>
-    <collision>
-      <origin xyz="0.0077 0.0001 -0.0234" rpy="-1.5708 -5.55112e-17 -1.38213e-14"/>
+      <origin xyz="0.0077 0.0001 -0.0234" rpy="-1.5708 -5.19179e-17 -1.66533e-16"/>
+      <geometry>
+        <mesh filename="package://so101_follower_description/meshes/sts3215_03a_v1.stl"/>
+      </geometry>
+      <material name="sts3215"/>
+    </visual>
+    <collision>
+      <origin xyz="0.0077 0.0001 -0.0234" rpy="-1.5708 -5.19179e-17 -1.66533e-16"/>
       <geometry>
         <mesh filename="package://so101_follower_description/meshes/sts3215_03a_v1.stl"/>
@@ -277,19 +270,34 @@
     <!-- Part wrist_roll_follower_so101_v1 -->
     <visual>
-      <origin xyz="5.55112e-17 -0.000218214 0.000949706" rpy="-3.14159 -5.55112e-17 -9.17912e-24"/>
-      <geometry>
-        <mesh filename="package://so101_follower_description/meshes/wrist_roll_follower_so101_v1.stl" scale="0.001 0.001 0.001"/>
-      </geometry>
-      <material name="3d_printed"/>
-    </visual>
-    <collision>
-      <origin xyz="5.55112e-17 -0.000218214 0.000949706" rpy="-3.14159 -5.55112e-17 -9.17912e-24"/>
-      <geometry>
-        <mesh filename="package://so101_follower_description/meshes/wrist_roll_follower_so101_v1.stl" scale="0.001 0.001 0.001"/>
-      </geometry>
-    </collision>
-  </link>
-  <!-- Link jaw -->
-  <link name="jaw_link">
+      <origin xyz="8.32667e-17 -0.000218214 0.000949706" rpy="-3.14159 -5.55112e-17 0"/>
+      <geometry>
+        <mesh filename="package://so101_follower_description/meshes/wrist_roll_follower_so101_v1.stl"/>
+      </geometry>
+      <material name="3d_printed"/>
+    </visual>
+    <collision>
+      <origin xyz="8.32667e-17 -0.000218214 0.000949706" rpy="-3.14159 -5.55112e-17 0"/>
+      <geometry>
+        <mesh filename="package://so101_follower_description/meshes/wrist_roll_follower_so101_v1.stl"/>
+      </geometry>
+    </collision>
+  </link>
+  <!-- Gripper frame (dummy link + fixed joint) -->
+  <link name="gripper_frame_link">
+    <origin xyz="0 0 0" rpy="0 -0 0"/>
+    <inertial>
+      <origin xyz="0 0 0" rpy="0 0 0"/>
+      <mass value="1e-9"/>
+      <inertia ixx="0" ixy="0" ixz="0" iyy="0" iyz="0" izz="0"/>
+    </inertial>
+  </link>
+  <joint name="gripper_frame_joint" type="fixed">
+    <origin xyz="-0.0079 -0.000218121 -0.0981274" rpy="0 3.14159 0"/>
+    <parent link="gripper_link"/>
+    <child link="gripper_frame_link"/>
+    <axis xyz="0 0 0"/>
+  </joint>
+  <!-- Link moving_jaw_so101_v1 -->
+  <link name="moving_jaw_so101_v1_link">
     <inertial>
       <origin xyz="-0.00157495 -0.0300244 0.0192755" rpy="0 0 0"/>
@@ -299,5 +307,5 @@
     <!-- Part moving_jaw_so101_v1 -->
     <visual>
-      <origin xyz="-5.55112e-17 -1.94746e-17 0.0189" rpy="9.53145e-17 -4.66093e-24 0"/>
+      <origin xyz="-5.55112e-17 -5.55112e-17 0.0189" rpy="9.53145e-17 6.93889e-18 1.24077e-24"/>
       <geometry>
         <mesh filename="package://so101_follower_description/meshes/moving_jaw_so101_v1.stl"/>
@@ -306,5 +314,5 @@
     </visual>
     <collision>
-      <origin xyz="-5.55112e-17 -1.94746e-17 0.0189" rpy="9.53145e-17 -4.66093e-24 0"/>
+      <origin xyz="-5.55112e-17 -5.55112e-17 0.0189" rpy="9.53145e-17 6.93889e-18 1.24077e-24"/>
       <geometry>
         <mesh filename="package://so101_follower_description/meshes/moving_jaw_so101_v1.stl"/>
@@ -312,11 +320,10 @@
     </collision>
   </link>
-  <!-- Joint from gripper to jaw -->
+  <!-- Joint from gripper to moving_jaw_so101_v1 -->
   <joint name="gripper" type="revolute">
-    <origin xyz="0.0202 0.0188 -0.0234" rpy="1.5708 -5.14108e-17 -1.38655e-14"/>
+    <origin xyz="0.0202 0.0188 -0.0234" rpy="1.5708 -5.24284e-08 -1.41553e-15"/>
     <parent link="gripper_link"/>
-    <child link="jaw_link"/>
-    <axis xyz="0 0 1"/>
-    <!-- calibrated limits: raw(2047,3489) home(2768) = (-1.110,+1.109) rad -->
+    <child link="moving_jaw_so101_v1_link"/>
+    <axis xyz="0 0 1"/>
     <limit effort="10" velocity="10" lower="-0.174533" upper="1.74533"/>
   </joint>
@@ -333,10 +340,9 @@
   <!-- Joint from wrist to gripper -->
   <joint name="wrist_roll" type="revolute">
-    <origin xyz="0 -0.0611 0.0181" rpy="1.5708 -9.38083e-08 3.14159"/>
+    <origin xyz="5.55112e-17 -0.0611 0.0181" rpy="1.5708 0.0486795 3.14159"/>
     <parent link="wrist_link"/>
     <child link="gripper_link"/>
     <axis xyz="0 0 1"/>
-    <!-- calibrated limits: raw(0,4766) home(2084) = (-3.194,+4.120) rad -->
-    <limit effort="10" velocity="10" lower="-3.194" upper="4.120"/>
+    <limit effort="10" velocity="10" lower="-2.74385" upper="2.84121"/>
   </joint>
   <transmission name="wrist_roll_trans">
@@ -352,10 +358,9 @@
   <!-- Joint from lower_arm to wrist -->
   <joint name="wrist_flex" type="revolute">
-    <origin xyz="-0.1349 0.0052 1.65232e-16" rpy="3.2474e-15 2.86219e-15 -1.5708"/>
+    <origin xyz="-0.1349 0.0052 3.62355e-17" rpy="4.02456e-15 8.67362e-16 -1.5708"/>
     <parent link="lower_arm_link"/>
     <child link="wrist_link"/>
     <axis xyz="0 0 1"/>
-    <!-- calibrated limits: raw(588,2917) home(1752) = (-1.786,+1.790) rad -->
-    <limit effort="10" velocity="10" lower="-1.786" upper="1.790"/>
+    <limit effort="10" velocity="10" lower="-1.65806" upper="1.65806"/>
   </joint>
   <transmission name="wrist_flex_trans">
@@ -370,11 +375,11 @@
   </transmission>
   <!-- Joint from upper_arm to lower_arm -->
+  <!-- Note: 5-degree calibration offset applied to joint limits -->
   <joint name="elbow_flex" type="revolute">
-    <origin xyz="-0.11257 -0.028 2.46331e-16" rpy="-1.22818e-15 5.75928e-16 1.5708"/>
+    <origin xyz="-0.11257 -0.028 1.73763e-16" rpy="-3.63608e-16 8.74301e-16 1.5708"/>
     <parent link="upper_arm_link"/>
     <child link="lower_arm_link"/>
     <axis xyz="0 0 1"/>
-    <!-- calibrated limits: raw(976,3130) home(2053) = (-1.653,+1.654) rad -->
-    <limit effort="10" velocity="10" lower="-1.653" upper="1.654"/>
+    <limit effort="10" velocity="10" lower="-1.69" upper="1.69"/>
   </joint>
   <transmission name="elbow_flex_trans">
@@ -394,6 +399,5 @@
     <child link="upper_arm_link"/>
     <axis xyz="0 0 1"/>
-    <!-- calibrated limits: raw(740,3370) home(2055) = (-2.018,+2.018) rad -->
-    <limit effort="10" velocity="10" lower="-2.018" upper="2.018"/>
+    <limit effort="10" velocity="10" lower="-1.74533" upper="1.74533"/>
   </joint>
   <transmission name="shoulder_lift_trans">
@@ -409,10 +413,9 @@
   <!-- Joint from base to shoulder -->
   <joint name="shoulder_pan" type="revolute">
-    <origin xyz="0.0207909 -0.0230745 0.0948817" rpy="-3.14159 6.03684e-16 1.5708"/>
+    <origin xyz="0.0388353 -8.97657e-09 0.0624" rpy="3.14159 4.18253e-17 -3.14159"/>
     <parent link="base_link"/>
     <child link="shoulder_link"/>
     <axis xyz="0 0 1"/>
-    <!-- calibrated limits: raw(745,3424) home(2084) = (-2.055,+2.058) rad -->
-    <limit effort="10" velocity="10" lower="-2.055" upper="2.058"/>
+    <limit effort="10" velocity="10" lower="-1.91986" upper="1.91986"/>
   </joint>
   <transmission name="shoulder_pan_trans">
@@ -426,3 +429,59 @@
     </actuator>
   </transmission>
+  <!-- Link wrist_camera_mount -->
+  <link name="wrist_camera_mount_link">
+    <inertial>
+      <origin xyz="0 0 0" rpy="0 0 0"/>
+      <mass value="0.02"/>
+      <inertia ixx="1e-5" ixy="0" ixz="0" iyy="1e-5" iyz="0" izz="1e-5"/>
+    </inertial>
+    <!-- Part wrist_camera_mount_so101_v1 (Hex-Nut Recess, 32x32 UVC module form factor) -->
+    <visual>
+      <origin xyz="0 0 0" rpy="0 0 0"/>
+      <geometry>
+        <mesh filename="package://so101_follower_description/meshes/wrist_camera_mount_so101_v1.stl" scale="0.001 0.001 0.001"/>
+      </geometry>
+      <material name="3d_printed"/>
+    </visual>
+    <collision>
+      <origin xyz="0 0 0" rpy="0 0 0"/>
+      <geometry>
+        <mesh filename="package://so101_follower_description/meshes/wrist_camera_mount_so101_v1.stl" scale="0.001 0.001 0.001"/>
+      </geometry>
+    </collision>
+  </link>
+  <!-- Link wrist_camera -->
+  <link name="wrist_camera_link">
+    <inertial>
+      <origin xyz="0 0 0" rpy="0 0 0"/>
+      <mass value="0.015"/>
+      <inertia ixx="1e-5" ixy="0" ixz="0" iyy="1e-5" iyz="0" izz="1e-5"/>
+    </inertial>
+    <!-- Part wrist_camera_so101_v1 -->
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