Commit message: Configure robot namespacing

File: hiwonder_ros2/so101_description/urdf/so101_macro.xacro (robot description, xacro)
@@ -3,6 +3,6 @@
 <!-- Onshape https://cad.onshape.com/documents/7715cc284bb430fe6dab4ffd/w/4fd0791b683777b02f8d975a/e/826c553ede3b7592eb9ca800 -->
 <!-- Derived from so101_new_calib.urdf: adds wrist camera mount + wrist camera (Hex-Nut 32x32 UVC module form factor) -->
-<robot xmlns:xacro="http://www.ros.org/wiki/xacro" name="so101_follower">
-  <xacro:macro name="so101_follower">
+<robot xmlns:xacro="http://www.ros.org/wiki/xacro" name="so101" params="prefix">
+  <xacro:macro name="so101" params="prefix">
     <!-- Materials -->
     <material name="3d_printed">
@@ -13,5 +13,5 @@
     </material>
     <!-- Link base -->
-    <link name="base_link">
+    <link name="${prefix}base_link">
       <inertial>
         <origin xyz="0.0137179 -5.19711e-05 0.0334843" rpy="0 0 0"/>
@@ -23,5 +23,5 @@
         <origin xyz="-0.00636471 -9.94414e-05 -0.0024" rpy="1.5708 -1.67685e-15 1.5708"/>
         <geometry>
-          <mesh filename="package://so101_follower_description/meshes/base_motor_holder_so101_v1.stl"/>
+          <mesh filename="package://so101_description/meshes/base_motor_holder_so101_v1.stl"/>
         </geometry>
         <material name="3d_printed"/>
@@ -30,5 +30,5 @@
         <origin xyz="-0.00636471 -9.94414e-05 -0.0024" rpy="1.5708 -1.67685e-15 1.5708"/>
         <geometry>
-          <mesh filename="package://so101_follower_description/meshes/base_motor_holder_so101_v1.stl"/>
+          <mesh filename="package://so101_description/meshes/base_motor_holder_so101_v1.stl"/>
         </geometry>
       </collision>
@@ -37,5 +37,5 @@
         <origin xyz="-0.00636471 -8.97657e-09 -0.0024" rpy="1.5708 -2.78073e-29 1.5708"/>
         <geometry>
-          <mesh filename="package://so101_follower_description/meshes/base_so101_v2.stl"/>
+          <mesh filename="package://so101_description/meshes/base_so101_v2.stl"/>
         </geometry>
         <material name="3d_printed"/>
@@ -44,5 +44,5 @@
         <origin xyz="-0.00636471 -8.97657e-09 -0.0024" rpy="1.5708 -2.78073e-29 1.5708"/>
         <geometry>
-          <mesh filename="package://so101_follower_description/meshes/base_so101_v2.stl"/>
+          <mesh filename="package://so101_description/meshes/base_so101_v2.stl"/>
         </geometry>
       </collision>
@@ -51,5 +51,5 @@
         <origin xyz="0.0263353 -8.97657e-09 0.0437" rpy="-8.21148e-16 7.84513e-18 1.249e-15"/>
         <geometry>
-          <mesh filename="package://so101_follower_description/meshes/sts3215_03a_v1.stl"/>
+          <mesh filename="package://so101_description/meshes/sts3215_03a_v1.stl"/>
         </geometry>
         <material name="sts3215"/>
@@ -58,5 +58,5 @@
         <origin xyz="0.0263353 -8.97657e-09 0.0437" rpy="-8.21148e-16 7.84513e-18 1.249e-15"/>
         <geometry>
-          <mesh filename="package://so101_follower_description/meshes/sts3215_03a_v1.stl"/>
+          <mesh filename="package://so101_description/meshes/sts3215_03a_v1.stl"/>
         </geometry>
       </collision>
@@ -65,5 +65,5 @@
         <origin xyz="-0.0309827 -0.000199441 0.0474" rpy="1.5708 -1.35493e-14 1.5708"/>
         <geometry>
-          <mesh filename="package://so101_follower_description/meshes/waveshare_mounting_plate_so101_v2.stl"/>
+          <mesh filename="package://so101_description/meshes/waveshare_mounting_plate_so101_v2.stl"/>
         </geometry>
         <material name="3d_printed"/>
@@ -72,10 +72,10 @@
         <origin xyz="-0.0309827 -0.000199441 0.0474" rpy="1.5708 -1.35493e-14 1.5708"/>
         <geometry>
-          <mesh filename="package://so101_follower_description/meshes/waveshare_mounting_plate_so101_v2.stl"/>
+          <mesh filename="package://so101_description/meshes/waveshare_mounting_plate_so101_v2.stl"/>
         </geometry>
       </collision>
     </link>
     <!-- Link shoulder -->
-    <link name="shoulder_link">
+    <link name="${prefix}shoulder_link">
       <inertial>
         <origin xyz="-0.0307604 -1.66727e-05 -0.0252713" rpy="0 0 0"/>
@@ -87,5 +87,5 @@
         <origin xyz="-0.0303992 0.000422241 -0.0417" rpy="1.5708 1.5708 0"/>
         <geometry>
-          <mesh filename="package://so101_follower_description/meshes/sts3215_03a_v1.stl"/>
+          <mesh filename="package://so101_description/meshes/sts3215_03a_v1.stl"/>
         </geometry>
         <material name="sts3215"/>
@@ -94,5 +94,5 @@
         <origin xyz="-0.0303992 0.000422241 -0.0417" rpy="1.5708 1.5708 0"/>
         <geometry>
-          <mesh filename="package://so101_follower_description/meshes/sts3215_03a_v1.stl"/>
+          <mesh filename="package://so101_description/meshes/sts3215_03a_v1.stl"/>
         </geometry>
       </collision>
@@ -101,5 +101,5 @@
         <origin xyz="-0.0675992 -0.000177759 0.0158499" rpy="1.5708 -1.5708 0"/>
         <geometry>
-          <mesh filename="package://so101_follower_description/meshes/motor_holder_so101_base_v1.stl"/>
+          <mesh filename="package://so101_description/meshes/motor_holder_so101_base_v1.stl"/>
         </geometry>
         <material name="3d_printed"/>
@@ -108,5 +108,5 @@
         <origin xyz="-0.0675992 -0.000177759 0.0158499" rpy="1.5708 -1.5708 0"/>
         <geometry>
-          <mesh filename="package://so101_follower_description/meshes/motor_holder_so101_base_v1.stl"/>
+          <mesh filename="package://so101_description/meshes/motor_holder_so101_base_v1.stl"/>
         </geometry>
       </collision>
@@ -115,5 +115,5 @@
         <origin xyz="0.0122008 2.22413e-05 0.0464" rpy="-1.5708 2.35221e-33 0"/>
         <geometry>
-          <mesh filename="package://so101_follower_description/meshes/rotation_pitch_so101_v1.stl"/>
+          <mesh filename="package://so101_description/meshes/rotation_pitch_so101_v1.stl"/>
         </geometry>
         <material name="3d_printed"/>
@@ -122,10 +122,10 @@
         <origin xyz="0.0122008 2.22413e-05 0.0464" rpy="-1.5708 2.35221e-33 0"/>
         <geometry>
-          <mesh filename="package://so101_follower_description/meshes/rotation_pitch_so101_v1.stl"/>
+          <mesh filename="package://so101_description/meshes/rotation_pitch_so101_v1.stl"/>
         </geometry>
       </collision>
     </link>
     <!-- Link upper_arm -->
-    <link name="upper_arm_link">
+    <link name="${prefix}upper_arm_link">
       <inertial>
         <origin xyz="-0.0898471 -0.00838224 0.0184089" rpy="0 0 0"/>
@@ -137,5 +137,5 @@
         <origin xyz="-0.11257 -0.0155 0.0187" rpy="-3.14159 -5.27356e-16 -1.5708"/>
         <geometry>
-          <mesh filename="package://so101_follower_description/meshes/sts3215_03a_v1.stl"/>
+          <mesh filename="package://so101_description/meshes/sts3215_03a_v1.stl"/>
         </geometry>
         <material name="sts3215"/>
@@ -144,5 +144,5 @@
         <origin xyz="-0.11257 -0.0155 0.0187" rpy="-3.14159 -5.27356e-16 -1.5708"/>
         <geometry>
-          <mesh filename="package://so101_follower_description/meshes/sts3215_03a_v1.stl"/>
+          <mesh filename="package://so101_description/meshes/sts3215_03a_v1.stl"/>
         </geometry>
       </collision>
@@ -151,5 +151,5 @@
         <origin xyz="-0.065085 0.012 0.0182" rpy="3.14159 -0 -1.30911e-30"/>
         <geometry>
-          <mesh filename="package://so101_follower_description/meshes/upper_arm_so101_v1.stl"/>
+          <mesh filename="package://so101_description/meshes/upper_arm_so101_v1.stl"/>
         </geometry>
         <material name="3d_printed"/>
@@ -158,10 +158,10 @@
         <origin xyz="-0.065085 0.012 0.0182" rpy="3.14159 -0 -1.30911e-30"/>
         <geometry>
-          <mesh filename="package://so101_follower_description/meshes/upper_arm_so101_v1.stl"/>
+          <mesh filename="package://so101_description/meshes/upper_arm_so101_v1.stl"/>
         </geometry>
       </collision>
     </link>
     <!-- Link lower_arm -->
-    <link name="lower_arm_link">
+    <link name="${prefix}lower_arm_link">
       <inertial>
         <origin xyz="-0.0980701 0.00324376 0.0182831" rpy="0 0 0"/>
@@ -173,5 +173,5 @@
         <origin xyz="-0.0648499 -0.032 0.0182" rpy="3.14159 -0 6.67202e-31"/>
         <geometry>
-          <mesh filename="package://so101_follower_description/meshes/under_arm_so101_v1.stl"/>
+          <mesh filename="package://so101_description/meshes/under_arm_so101_v1.stl"/>
         </geometry>
         <material name="3d_printed"/>
@@ -180,5 +180,5 @@
         <origin xyz="-0.0648499 -0.032 0.0182" rpy="3.14159 -0 6.67202e-31"/>
         <geometry>
-          <mesh filename="package://so101_follower_description/meshes/under_arm_so101_v1.stl"/>
+          <mesh filename="package://so101_description/meshes/under_arm_so101_v1.stl"/>
         </geometry>
       </collision>
@@ -187,5 +187,5 @@
         <origin xyz="-0.0648499 -0.032 0.018" rpy="-3.14159 -2.55351e-15 -1.83387e-30"/>
         <geometry>
-          <mesh filename="package://so101_follower_description/meshes/motor_holder_so101_wrist_v1.stl"/>
+          <mesh filename="package://so101_description/meshes/motor_holder_so101_wrist_v1.stl"/>
         </geometry>
         <material name="3d_printed"/>
@@ -194,5 +194,5 @@
         <origin xyz="-0.0648499 -0.032 0.018" rpy="-3.14159 -2.55351e-15 -1.83387e-30"/>
         <geometry>
-          <mesh filename="package://so101_follower_description/meshes/motor_holder_so101_wrist_v1.stl"/>
+          <mesh filename="package://so101_description/meshes/motor_holder_so101_wrist_v1.stl"/>
         </geometry>
       </collision>
@@ -201,5 +201,5 @@
         <origin xyz="-0.1224 0.0052 0.0187" rpy="-3.14159 -7.88861e-31 -3.14159"/>
         <geometry>
-          <mesh filename="package://so101_follower_description/meshes/sts3215_03a_v1.stl"/>
+          <mesh filename="package://so101_description/meshes/sts3215_03a_v1.stl"/>
         </geometry>
         <material name="sts3215"/>
@@ -208,10 +208,10 @@
         <origin xyz="-0.1224 0.0052 0.0187" rpy="-3.14159 -7.88861e-31 -3.14159"/>
         <geometry>
-          <mesh filename="package://so101_follower_description/meshes/sts3215_03a_v1.stl"/>
+          <mesh filename="package://so101_description/meshes/sts3215_03a_v1.stl"/>
         </geometry>
       </collision>
     </link>
     <!-- Link wrist -->
-    <link name="wrist_link">
+    <link name="${prefix}wrist_link">
       <inertial>
         <origin xyz="-0.000103312 -0.0386143 0.0281156" rpy="0 0 0"/>
@@ -223,5 +223,5 @@
         <origin xyz="8.32667e-17 -0.0424 0.0306" rpy="1.5708 1.5708 0"/>
         <geometry>
-          <mesh filename="package://so101_follower_description/meshes/sts3215_03a_no_horn_v1.stl"/>
+          <mesh filename="package://so101_description/meshes/sts3215_03a_no_horn_v1.stl"/>
         </geometry>
         <material name="3d_printed"/>
@@ -230,5 +230,5 @@
         <origin xyz="8.32667e-17 -0.0424 0.0306" rpy="1.5708 1.5708 0"/>
         <geometry>
-          <mesh filename="package://so101_follower_description/meshes/sts3215_03a_no_horn_v1.stl"/>
+          <mesh filename="package://so101_description/meshes/sts3215_03a_no_horn_v1.stl"/>
         </geometry>
       </collision>
@@ -237,5 +237,5 @@
         <origin xyz="0 -0.028 0.0181" rpy="-1.5708 -1.5708 0"/>
         <geometry>
-          <mesh filename="package://so101_follower_description/meshes/wrist_roll_pitch_so101_v2.stl"/>
+          <mesh filename="package://so101_description/meshes/wrist_roll_pitch_so101_v2.stl"/>
         </geometry>
         <material name="3d_printed"/>
@@ -244,10 +244,10 @@
         <origin xyz="0 -0.028 0.0181" rpy="-1.5708 -1.5708 0"/>
         <geometry>
-          <mesh filename="package://so101_follower_description/meshes/wrist_roll_pitch_so101_v2.stl"/>
+          <mesh filename="package://so101_description/meshes/wrist_roll_pitch_so101_v2.stl"/>
         </geometry>
       </collision>
     </link>
     <!-- Link gripper -->
-    <link name="gripper_link">
+    <link name="${prefix}gripper_link">
       <inertial>
         <origin xyz="0.000213627 0.000245138 -0.025187" rpy="0 0 0"/>
@@ -259,5 +259,5 @@
         <origin xyz="0.0077 0.0001 -0.0234" rpy="-1.5708 -5.19179e-17 -1.66533e-16"/>
         <geometry>
-          <mesh filename="package://so101_follower_description/meshes/sts3215_03a_v1.stl"/>
+          <mesh filename="package://so101_description/meshes/sts3215_03a_v1.stl"/>
         </geometry>
         <material name="sts3215"/>
@@ -266,5 +266,5 @@
         <origin xyz="0.0077 0.0001 -0.0234" rpy="-1.5708 -5.19179e-17 -1.66533e-16"/>
         <geometry>
-          <mesh filename="package://so101_follower_description/meshes/sts3215_03a_v1.stl"/>
+          <mesh filename="package://so101_description/meshes/sts3215_03a_v1.stl"/>
         </geometry>
       </collision>
@@ -273,5 +273,5 @@
         <origin xyz="8.32667e-17 -0.000218214 0.000949706" rpy="-3.14159 -5.55112e-17 0"/>
         <geometry>
-          <mesh filename="package://so101_follower_description/meshes/wrist_roll_follower_so101_v1.stl"/>
+          <mesh filename="package://so101_description/meshes/wrist_roll_follower_so101_v1.stl"/>
         </geometry>
         <material name="3d_printed"/>
@@ -280,10 +280,10 @@
         <origin xyz="8.32667e-17 -0.000218214 0.000949706" rpy="-3.14159 -5.55112e-17 0"/>
         <geometry>
-          <mesh filename="package://so101_follower_description/meshes/wrist_roll_follower_so101_v1.stl"/>
+          <mesh filename="package://so101_description/meshes/wrist_roll_follower_so101_v1.stl"/>
         </geometry>
       </collision>
     </link>
     <!-- Gripper frame (dummy link + fixed joint) -->
-    <link name="gripper_frame_link">
+    <link name="${prefix}gripper_frame_link">
       <origin xyz="0 0 0" rpy="0 -0 0"/>
       <inertial>
@@ -293,12 +293,12 @@
       </inertial>
     </link>
-    <joint name="gripper_frame_joint" type="fixed">
+    <joint name="${prefix}gripper_frame_joint" type="fixed">
       <origin xyz="-0.0079 -0.000218121 -0.0981274" rpy="0 3.14159 0"/>
-      <parent link="gripper_link"/>
-      <child link="gripper_frame_link"/>
+      <parent link="${prefix}gripper_link"/>
+      <child link="${prefix}gripper_frame_link"/>
       <axis xyz="0 0 0"/>
     </joint>
     <!-- Link moving_jaw_so101_v1 -->
-    <link name="moving_jaw_so101_v1_link">
+    <link name="${prefix}moving_jaw_so101_v1_link">
       <inertial>
         <origin xyz="-0.00157495 -0.0300244 0.0192755" rpy="0 0 0"/>
@@ -310,5 +310,5 @@
         <origin xyz="-5.55112e-17 -5.55112e-17 0.0189" rpy="9.53145e-17 6.93889e-18 1.24077e-24"/>
         <geometry>
-          <mesh filename="package://so101_follower_description/meshes/moving_jaw_so101_v1.stl"/>
+          <mesh filename="package://so101_description/meshes/moving_jaw_so101_v1.stl"/>
         </geometry>
         <material name="3d_printed"/>
@@ -317,5 +317,5 @@
         <origin xyz="-5.55112e-17 -5.55112e-17 0.0189" rpy="9.53145e-17 6.93889e-18 1.24077e-24"/>
         <geometry>
-          <mesh filename="package://so101_follower_description/meshes/moving_jaw_so101_v1.stl"/>
+          <mesh filename="package://so101_description/meshes/moving_jaw_so101_v1.stl"/>
         </geometry>
       </collision>
@@ -324,6 +324,6 @@
     <joint name="gripper" type="revolute">
       <origin xyz="0.0202 0.0188 -0.0234" rpy="1.5708 -5.24284e-08 -1.41553e-15"/>
-      <parent link="gripper_link"/>
-      <child link="moving_jaw_so101_v1_link"/>
+      <parent link="${prefix}gripper_link"/>
+      <child link="${prefix}moving_jaw_so101_v1_link"/>
       <axis xyz="0 0 1"/>
       <limit effort="10" velocity="10" lower="-0.174533" upper="1.74533"/>
@@ -332,6 +332,6 @@
     <joint name="wrist_roll" type="revolute">
       <origin xyz="5.55112e-17 -0.0611 0.0181" rpy="1.5708 0.0486795 3.14159"/>
-      <parent link="wrist_link"/>
-      <child link="gripper_link"/>
+      <parent link="${prefix}wrist_link"/>
+      <child link="${prefix}gripper_link"/>
       <axis xyz="0 0 1"/>
       <limit effort="10" velocity="10" lower="-2.74385" upper="2.84121"/>
@@ -340,6 +340,6 @@
     <joint name="wrist_flex" type="revolute">
       <origin xyz="-0.1349 0.0052 3.62355e-17" rpy="4.02456e-15 8.67362e-16 -1.5708"/>
-      <parent link="lower_arm_link"/>
-      <child link="wrist_link"/>
+      <parent link="${prefix}lower_arm_link"/>
+      <child link="${prefix}wrist_link"/>
       <axis xyz="0 0 1"/>
       <limit effort="10" velocity="10" lower="-1.65806" upper="1.65806"/>
@@ -349,6 +349,6 @@
     <joint name="elbow_flex" type="revolute">
       <origin xyz="-0.11257 -0.028 1.73763e-16" rpy="-3.63608e-16 8.74301e-16 1.5708"/>
-      <parent link="upper_arm_link"/>
-      <child link="lower_arm_link"/>
+      <parent link="${prefix}upper_arm_link"/>
+      <child link="${prefix}lower_arm_link"/>
       <axis xyz="0 0 1"/>
       <limit effort="10" velocity="10" lower="-1.69" upper="1.69"/>
@@ -357,6 +357,6 @@
     <joint name="shoulder_lift" type="revolute">
       <origin xyz="-0.0303992 -0.0182778 -0.0542" rpy="-1.5708 -1.5708 0"/>
-      <parent link="shoulder_link"/>
-      <child link="upper_arm_link"/>
+      <parent link="${prefix}shoulder_link"/>
+      <child link="${prefix}upper_arm_link"/>
       <axis xyz="0 0 1"/>
       <limit effort="10" velocity="10" lower="-1.74533" upper="1.74533"/>
@@ -365,11 +365,11 @@
     <joint name="shoulder_pan" type="revolute">
       <origin xyz="0.0388353 -8.97657e-09 0.0624" rpy="3.14159 4.18253e-17 -3.14159"/>
-      <parent link="base_link"/>
-      <child link="shoulder_link"/>
+      <parent link="${prefix}base_link"/>
+      <child link="${prefix}shoulder_link"/>
       <axis xyz="0 0 1"/>
       <limit effort="10" velocity="10" lower="-1.91986" upper="1.91986"/>
     </joint>
     <!-- Link wrist_camera_mount -->
-    <link name="wrist_camera_mount_link">
+    <link name="${prefix}wrist_camera_mount_link">
       <inertial>
         <origin xyz="0 0 0" rpy="0 0 0"/>
@@ -381,17 +381,17 @@
         <origin xyz="0 0 0" rpy="0 0 0"/>
         <geometry>
-          <mesh filename="package://so101_follower_description/meshes/wrist_camera_mount_so101_v1.stl" scale="0.001 0.001 0.001"/>
-        </geometry>
-        <material name="3d_printed"/>
-      </visual>
-      <collision>
-        <origin xyz="0 0 0" rpy="0 0 0"/>
-        <geometry>
-          <mesh filename="package://so101_follower_description/meshes/wrist_camera_mount_so101_v1.stl" scale="0.001 0.001 0.001"/>
+          <mesh filename="package://so101_description/meshes/wrist_camera_mount_so101_v1.stl" scale="0.001 0.001 0.001"/>
+        </geometry>
+        <material name="3d_printed"/>
+      </visual>
+      <collision>
+        <origin xyz="0 0 0" rpy="0 0 0"/>
+        <geometry>
+          <mesh filename="package://so101_description/meshes/wrist_camera_mount_so101_v1.stl" scale="0.001 0.001 0.001"/>
         </geometry>
       </collision>
     </link>
     <!-- Link wrist_camera -->
-    <link name="wrist_camera_link">
+    <link name="${prefix}wrist_camera_link">
       <inertial>
         <origin xyz="0 0 0" rpy="0 0 0"/>
@@ -403,26 +403,26 @@
         <origin xyz="0 0 0" rpy="0 0 0"/>
         <geometry>
-          <mesh filename="package://so101_follower_description/meshes/wrist_camera_so101_v1.stl"/>
-        </geometry>
-        <material name="3d_printed"/>
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
File: hiwonder_ros2/so101_description/urdf/so101_ros2_control.xacro (robot description, xacro)
@@ -1,9 +1,9 @@
 <?xml version="1.0"?>
 <robot xmlns:xacro="http://www.ros.org/wiki/xacro">
-  <xacro:macro name="so101_follower_ros2_control" params="port calibration_file">
-    <ros2_control name="so101_follower" type="system">
+  <xacro:macro name="so101_ros2_control" params="port calibration_file prefix robot_plugin">
+    <ros2_control name="${prefix}so101" type="system">
       <hardware>
         <plugin>lerobot_ros2_control/LeRobotSystemHardware</plugin>
-        <param name="robot_plugin">hiwonder_lerobot_cpp/Follower</param>
+        <param name="robot_plugin">${robot_plugin}</param>
         <param name="port">${port}</param>
         <param name="baud_rate">1000000</param>
